File: stm32f103_fc.brd (EAGLE design)
At the start: 59.4 x 80 mm, 48 parts, among them IC1 STM32F10XCXT6, IC2 LD117AS33TR, J5 1X2-3.5MM, J6 1X2-3.5MM, U2 9DoF IMU, Y1 8MHz, Y2 32.768MHz

Commit message: BOM next
Parts:
- removed J5: 1X2-3.5MM, adafruit:1X2-3.5MM
- added PYRO2: 1X2-3.5MM, adafruit:1X2-3.5MM
- Q1, Q2: device adafruit:TO220V -> adafruit:SOT23
- moved C9 10.9 mm to (61.0, 66.0)
- moved S1 3.81 mm to (48.3, 8.89)
- moved J3 2.84 mm to (61.0, 8.89), turned to 270 degrees
- renumbered J6 to PYRO1
Connections:
- net 5V: now also PYRO2.1; no longer J5.1
- net GND: now also Q1.2, Q2.2; no longer Q1.3, Q2.3
- net N$12: now also PYRO2.2; no longer J5.2
- net N$13: now also Q2.3; no longer Q2.2
- net N$15: now also Q1.3; no longer Q1.2
Routing:
- net GND: track 399.6 -> 369.6 mm, vias 8 -> 10
- net N$1: track 38.3 -> 24.7 mm, vias 1 -> 3
- net N$6: track 37.6 -> 28.7 mm, vias 0 -> 2
- net N$8: track 21.2 -> 12.8 mm
- net N$15: track 68.6 -> 75.7 mm, vias 1 -> 2
- net PB6: track 66.3 -> 72.0 mm, vias 2 -> 3
- net 5V: track 194.0 -> 189.3 mm
- net PB7: track 55.5 -> 60.0 mm
- net N$12: track 45.2 -> 42.6 mm
- net N$13: track 53.7 -> 51.1 mm, vias 1 -> 2
- net RESET: track 71.7 -> 69.9 mm
- net PB8: track 17.7 -> 19.0 mm
- net PA6: track 60.9 -> 61.6 mm
Other:
- board size 59.4 x 80 mm -> 55.5 x 74.9 mm

Commit message: relayout board
Parts:
- removed C15: 100nF, SparkFun-Capacitors:0805
- removed C22: 100nF, SparkFun-Capacitors:0603
- removed R14: 470ohm, SparkFun-Resistors:0603
- removed R7: 1.58ohm, SparkFun-Resistors:0603
- removed R8: 4.7k, SparkFun-Resistors:0603
- added C4, C8: 12pF, SparkFun-Capacitors:0603
- added R12, R15: 1omh, SparkFun-Resistors:0603
- C1: value 100nF -> 0.1uF
- C10, C16: value 20pF -> 100pF; device SparkFun-Capacitors:0805 -> SparkFun-Capacitors:0603
- C11, C13, C14, C7: value 100nF -> 0.1uF; device SparkFun-Capacitors:0805 -> SparkFun-Capacitors:0402
- C17, C18: value 20pF -> 0.1uF; device SparkFun-Capacitors:0805 -> SparkFun-Capacitors:0603
- C5: value 100nF -> 10nF; device SparkFun-Capacitors:0805 -> SparkFun-Capacitors:0603
- C6: value 10nF -> 0.1uF; device SparkFun-Capacitors:0805 -> SparkFun-Capacitors:0402
- C9: device SparkFun-Capacitors:0805 -> SparkFun-Capacitors:0603
- IC2: value LD117AS33TR -> LD1117AS33TR
- R1, R2: value 1k -> 100k
- R10, R13: value 1ohm -> 22
- R11: value 470ohm -> 680
- R3: value 70ohm -> 10k
- R4: value 70ohm -> 470
- R5: value 10k -> 470
- R6: value 1.58ohm -> 10k
- R9: value 1M -> 680
- moved C7 55.8 mm to (39.4, 67.3)
- moved R13 42.4 mm to (58.4, 21.6)
- moved R10 37.1 mm to (58.4, 25.4)
- moved R3 36.9 mm to (30.5, 52.1)
- moved C18 34.5 mm to (27.9, 39.4)
- moved R11 31.1 mm to (52.1, 54.6)
- moved C11 31.0 mm to (66.0, 73.7)
- moved C13 30.5 mm to (66.0, 69.8)
- moved C10 27.9 mm to (27.9, 62.2)
- moved C6 26.9 mm to (35.6, 27.9), turned to 180 degrees
- moved C1 25.0 mm to (30.5, 48.3)
- moved R1 24.0 mm to (71.1, 19.1)
- moved R4 23.7 mm to (39.4, 52.1)
- moved Y1 23.3 mm to (48.3, 26.7), turned to 180 degrees
- moved R9 23.2 mm to (62.2, 58.4)
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Connections:
- net 5V: now also R6.1; no longer R8.1
- net BOOT0: now also R1.1; no longer R2.1
- net BOOT1: now also R2.2; no longer R1.2
- net GND: now also C10.2, C11.2, C13.2, C14.2, C16.2, C6.1, C7.2, R4.1, R5.1; no longer C11.1, C13.1, C14.1, C15.1, C22.2, C6.2, C7.1, R11.1, R14.1
- net N$1: now also R1.2; no longer R2.2
- net N$10: now also C4.2, C8.2; no longer C10.2, C16.2
- net N$11: now also C6.2; no longer C7.2
- net N$12: now also R15.2; no longer R13.1
- net N$13: now also R15.1; no longer R13.2
- net N$14: now also R12.2; no longer R10.1
- net N$15: now also R12.1; no longer R10.2
- net N$2: now also R2.1; no longer R1.1
- net N$3: now also R9.2; no longer R3.2
- net N$5: now also R11.2; no longer R4.2
- net N$6: now also R10.1; no longer R6.1
- net N$7: now also C4.1; no longer C10.1, R9.2
- net N$8: now also R13.1; no longer R7.1
- net N$9: now also C8.1; no longer C16.1, R9.1
- net PA11: now also R10.2; no longer R6.2
- net PA12: now also R13.2, R6.2; no longer R7.2, R8.2
- net PB6: now also R5.2; no longer R14.2
- net PB7: now also R4.2; no longer R11.2
- net PC14: now also C10.1; no longer C18.1
- net PC15: now also C16.1; no longer C17.1
- net RESET: now also R3.1; no longer R5.1
- net VCC3V3: now also C11.1, C13.1, C14.1, C17.1, C18.1, C7.1, R11.1, R3.2, R9.1; no longer C11.2, C13.2, C14.2, C15.2, C22.1, C6.1, R3.1, R4.1, R5.2
Routing:
- net PC14: track 36.9 -> 107.4 mm, vias 1 -> 2
- net RESET: track 69.9 -> 129.6 mm, vias 0 -> 2
- net PB7: track 60.0 -> 110.6 mm
- net BOOT0: track 29.2 -> 77.5 mm, vias 2 -> 6
- net PA12: track 95.9 -> 62.0 mm, vias 2 -> 7
- net N$12: track 42.6 -> 8.81 mm
- net N$15: track 75.7 -> 42.6 mm
- net BOOT1: track 7.07 -> 34.3 mm, vias 2 -> 0
- net N$10: track 29.0 -> 3.85 mm, vias 2 -> 0
- net N$14: track 32.7 -> 11.8 mm
- net SWDIO: track 31.1 -> 50.6 mm, vias 0 -> 2
- net 5V: track 189.3 -> 205.8 mm
- net N$5: track 21.8 -> 6.21 mm
- net PC15: track 66.2 -> 51.3 mm, vias 1 -> 3
- net N$13: track 51.1 -> 63.7 mm, vias 2 -> 0
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
Commit message: done version 2
Parts:
- moved R15 66.0 mm to (58.4, 68.6), turned to 0 degrees
- moved R12 62.7 mm to (58.4, 72.4), turned to 0 degrees
- moved C11 56.4 mm to (10.2, 81.3), turned to 270 degrees
- moved D1 55.4 mm to (10.2, 69.8), turned to 270 degrees
- moved R9 54.3 mm to (10.2, 73.7), turned to 270 degrees
- moved Q1 52.3 mm to (50.8, 72.4)
- moved C3 46.7 mm to (53.3, 83.8), turned to 270 degrees
- moved C13 45.6 mm to (21.6, 80.0), turned to 270 degrees
- moved Q2 43.3 mm to (50.8, 68.6)
- moved PYRO2 42.3 mm to (63.5, 36.8), turned to 270 degrees
- moved R6 40.7 mm to (25.4, 27.9), turned to 180 degrees
- moved C4 39.4 mm to (40.6, 33.0)
- moved U2 39.4 mm to (26.7, 61.0)
- moved C8 37.5 mm to (45.7, 33.0), turned to 180 degrees
- moved C17 37.5 mm to (61.0, 61.0), turned to 270 degrees
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Routing:
- net RESET: track 129.6 -> 40.4 mm, vias 2 -> 0
- net PC14: track 107.4 -> 18.6 mm, vias 2 -> 0
- net PB7: track 110.6 -> 43.6 mm
- net N$13: track 63.7 -> 7.87 mm
- net BOOT0: track 77.5 -> 22.8 mm, vias 6 -> 2
- net PB6: track 77.0 -> 30.0 mm, vias 3 -> 2
- net PA6: track 68.8 -> 22.0 mm, vias 1 -> 0
- net N$7: track 60.7 -> 14.4 mm, vias 3 -> 0
- net N$9: track 57.3 -> 14.8 mm, vias 3 -> 0
- net N$14: track 11.8 -> 51.5 mm, vias 0 -> 2
- net VCC3V3: track 207.3 -> 240.2 mm, vias 4 -> 8
- net N$15: track 42.6 -> 10.5 mm
- net N$12: track 8.81 -> 39.8 mm, vias 0 -> 2
- net PC15: track 51.3 -> 22.4 mm, vias 3 -> 0
- net SWDIO: track 50.6 -> 22.6 mm
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- removed copper zone on layer 1, net GND
Other:
- board size 55.5 x 74.9 mm -> 64.4 x 87.6 mm
- board text added: "SPACE PIRATE V1.0.0"
- board text removed: "Space Pirate v1.0.0"

Commit message: done version 2
Parts:
- moved D1 9.25 mm to (19.1, 67.3)
- moved C11 8.52 mm to (17.8, 85.1)
- moved R9 6.35 mm to (16.5, 73.7)
Routing:
- net VCC3V3: track 240.2 -> 232.6 mm
- net N$3: track 2.08 -> 5.68 mm
- net GND: track 356.9 -> 354.0 mm, vias 21 -> 20
Other:
- board size 64.4 x 87.6 mm -> 60.6 x 87.6 mm

Commit message: done version 2
Parts:
- moved C11 22.5 mm to (39.4, 78.7)
- moved C7 14.0 mm to (27.9, 80.0)
- moved R9 10.2 mm to (26.7, 72.4)
- moved D1 7.73 mm to (26.7, 68.6)
- moved C9 2.54 mm to (57.1, 83.8)
- moved POWER_INPUT 1.27 mm to (63.5, 82.5)
Routing:
- net GND: track 354.0 -> 343.3 mm, vias 20 -> 19
- net VCC3V3: track 232.6 -> 223.8 mm, vias 8 -> 9
- net N$3: track 5.68 -> 2.08 mm
- net 5V: track 182.3 -> 180.3 mm
- added copper zone on layer 1, net GND
Other:
- board size 60.6 x 87.6 mm -> 53 x 78.7 mm

Commit message: done version 2
Routing:
- net GND: track 343.3 -> 339.4 mm
- net VCC3V3: track 223.8 -> 221.3 mm, vias 9 -> 7

Commit message: done
Parts:
- moved IC2 2.77 mm to (43.2, 81.1)
- moved C3 2.61 mm to (51.6, 81.9)
- moved C9 2.12 mm to (58.0, 81.9)
- moved C11 1.96 mm to (37.4, 79.0)
- moved POWER_INPUT 1.48 mm to (63.5, 81.1)
- moved C14 0.88 mm to (34.7, 79.9)
Routing:
- net GND: track 339.4 -> 293.0 mm
- net VCC3V3: track 221.3 -> 232.1 mm, vias 7 -> 9
- net 5V: track 180.3 -> 184.9 mm
- net PA11: track 49.3 -> 51.8 mm
- net PB7: track 43.9 -> 42.1 mm
- net N$8: track 11.3 -> 10.5 mm
- net PA12: track 54.9 -> 55.5 mm
- net RESET: track 40.4 -> 41.0 mm
- net PB6: track 29.8 -> 29.2 mm
Other:
- board size 53 x 78.7 mm -> 53.1 x 76.5 mm

Commit message: done final cam
Routing:
- net VCC3V3: track 232.1 -> 231.0 mm
- net GND: track 293.0 -> 292.5 mm
Changed lines of the file:
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@@
 <wire x1="29.235909375" y1="83.82" x2="26.4898625" y2="83.82" width="0.508" layer="1"/>
 <wire x1="26.4898625" y1="83.82" x2="25.4" y2="83.82" width="0.508" layer="1"/>
-<wire x1="44.45" y1="41.91" x2="49.53" y2="36.83" width="0.254" layer="1"/>
 <wire x1="49.53" y1="36.83" x2="49.53" y2="23.799221875" width="0.254" layer="1"/>
 <wire x1="49.53" y1="23.799221875" x2="47.320778125" y2="21.59" width="0.254" layer="1"/>
@@
 <via x="59.69" y="46.99" extent="1-16" drill="0.45"/>
 <wire x1="51.5076" y1="48.228790625" x2="49.5118875" y2="48.228790625" width="0.254" layer="1"/>
-<wire x1="44.45" y1="43.18" x2="44.463096875" y2="43.18" width="0.254" layer="1"/>
-<wire x1="44.463096875" y1="43.18" x2="49.5118875" y2="48.228790625" width="0.254" layer="1"/>
 <wire x1="59.69" y1="46.99" x2="59.69" y2="53.34" width="0.254" layer="16"/>
 <via x="59.69" y="53.34" extent="1-16" drill="0.45"/>
@@
 <wire x1="62.26586875" y1="55.91586875" x2="62.26586875" y2="60.986296875" width="0.254" layer="1"/>
 <wire x1="59.69" y1="53.34" x2="62.26586875" y2="55.91586875" width="0.254" layer="1"/>
-<wire x1="28.2225" y1="59.96" x2="28.226746875" y2="59.955753125" width="0.254" layer="1"/>
-<wire x1="28.226746875" y1="59.955753125" x2="30.496009375" y2="59.955753125" width="0.254" layer="1"/>
 <via x="30.496009375" y="59.955753125" extent="1-16" drill="0.45"/>
 <via x="33.23" y="46.5724" extent="1-16" drill="0.45"/>
 <wire x1="30.496009375" y1="59.955753125" x2="30.4828625" y2="59.94260625" width="0.254" layer="16"/>
 <wire x1="34.7076" y1="48.05" x2="33.23" y2="46.5724" width="0.254" layer="1"/>
-<wire x1="40.03" y1="81.0538625" x2="39.37" y2="80.3938625" width="0.254" layer="1"/>
 <via x="24.13" y="77.47" extent="1-16" drill="0.45"/>
 <wire x1="24.13" y1="77.47" x2="24.13" y2="78.16013125" width="0.254" layer="1"/>
@@
 <wire x1="59.69" y1="46.99" x2="52.746390625" y2="46.99" width="0.254" layer="1"/>
 <wire x1="52.746390625" y1="46.99" x2="51.5076" y2="48.228790625" width="0.254" layer="1"/>
-<wire x1="44.43" y1="43.2" x2="44.45" y2="43.18" width="0.2032" layer="1"/>
 <wire x1="38.68" y1="48.05" x2="41.692409375" y2="48.05" width="0.2032" layer="1"/>
 <wire x1="44.43" y1="46.3" x2="44.43" y2="47.47629375" width="0.2032" layer="1"/>
@@
 <wire x1="43.850553125" y1="48.055740625" x2="41.69815" y2="48.055740625" width="0.2032" layer="1"/>
 <wire x1="41.69815" y1="48.055740625" x2="41.692409375" y2="48.05" width="0.2032" layer="1"/>
-<wire x1="44.43" y1="41.93" x2="44.45" y2="41.91" width="0.2032" layer="1"/>
-<wire x1="44.45" y1="41.91" x2="44.45" y2="43.166903125" width="0.2032" layer="1"/>
-<wire x1="44.45" y1="43.166903125" x2="44.463096875" y2="43.18" width="0.2032" layer="1"/>
-<wire x1="44.45" y1="43.166903125" x2="44.45" y2="46.28" width="0.2032" layer="1"/>
 <wire x1="44.45" y1="46.28" x2="44.43" y2="46.3" width="0.2032" layer="1"/>
 <wire x1="25.4" y1="80.86" x2="25.4" y2="82.7301375" width="0.2032" layer="1"/>
@@
 <wire x1="34.683253125" y1="81.88143125" x2="36.621821875" y2="83.82" width="0.2032" layer="1"/>
 <wire x1="37.421675" y1="79.563440625" x2="37.421675" y2="80.8708375" width="0.2032" layer="1"/>
-<wire x1="37.421675" y1="80.8708375" x2="37.421675" y2="81.0538625" width="0.2032" layer="1"/>
 <wire x1="39.34419375" y1="83.82" x2="39.37" y2="83.79419375" width="0.2032" layer="1"/>
 <wire x1="38.68" y1="48.05" x2="34.7076" y2="48.05" width="0.254" layer="1"/>
@@
 <wire x1="29.70589375" y1="44.926615625" x2="28.36" y2="43.580721875" width="0.2032" layer="1"/>
 <wire x1="28.36" y1="43.580721875" x2="28.36" y2="43.18" width="0.2032" layer="1"/>
-<wire x1="37.421675" y1="80.8708375" x2="37.421675" y2="82.567471875" width="0.254" layer="1"/>
 <wire x1="37.421675" y1="82.567471875" x2="38.674203125" y2="83.82" width="0.254" layer="1"/>
 <wire x1="39.37" y1="83.79419375" x2="40.03" y2="83.13419375" width="0.508" layer="1"/>
 <wire x1="40.03" y1="83.13419375" x2="40.03" y2="81.0538625" width="0.508" layer="1"/>
+<wire x1="44.43" y1="46.3" x2="44.43" y2="46.28298125" width="0.254" layer="1"/>
+<wire x1="44.43" y1="46.28298125" x2="44.43" y2="46.2802625" width="0.254" layer="1"/>
+<wire x1="44.43" y1="46.2802625" x2="44.43" y2="43.657159375" width="0.254" layer="1"/>
+<wire x1="44.43" y1="43.657159375" x2="44.43" y2="41.93" width="0.254" layer="1"/>
+<wire x1="44.43" y1="41.93" x2="49.53" y2="36.83" width="0.254" layer="1"/>
+<wire x1="44.43" y1="46.28298125" x2="44.43298125" y2="46.28" width="0.254" layer="1"/>
+<wire x1="44.43298125" y1="46.28" x2="44.45" y2="46.28" width="0.254" layer="1"/>
+<wire x1="44.43" y1="46.2802625" x2="44.4302625" y2="46.28" width="0.254" layer="1"/>
+<wire x1="44.4302625" y1="46.28" x2="44.43298125" y2="46.28" width="0.254" layer="1"/>
+<wire x1="30.4917625" y1="59.96" x2="30.496009375" y2="59.955753125" width="0.254" layer="1"/>
+<wire x1="49.5118875" y1="48.228790625" x2="46.0432375" y2="44.760140625" width="0.2286" layer="1"/>
+<wire x1="46.0432375" y1="44.760140625" x2="45.106328125" y2="44.760140625" width="0.2286" layer="1"/>
+<wire x1="45.106328125" y1="44.760140625" x2="44.43" y2="44.0838125" width="0.2286" layer="1"/>
+<wire x1="44.43" y1="44.0838125" x2="44.43" y2="43.657159375" width="0.2286" layer="1"/>
+<wire x1="28.2225" y1="59.96" x2="30.4917625" y2="59.96" width="0.2286" layer="1"/>
+<wire x1="37.421675" y1="80.8708375" x2="37.421675" y2="82.567471875" width="0.2286" layer="1"/>
 </signal>
 <signal name="N$1">
@@
 <wire x1="47.68" y1="53.05" x2="45.575" y2="53.05" width="0.254" layer="1"/>
 <wire x1="45.575" y1="53.05" x2="45.575" y2="50.945" width="0.254" layer="1"/>
-<wire x1="26.67" y1="67.703" x2="27.063" y2="67.31" width="0.254" layer="1"/>
 <wire x1="27.94" y1="79.43" x2="27.94" y2="76.2" width="0.254" layer="1"/>
 <wire x1="37.421675" y1="78.403440625" x2="37.421675" y2="76.2" width="0.254" layer="1"/>
@@
 <contactref element="SERVO_X" pad="2"/>
 <contactref element="SERVO_Y" pad="2"/>
-<wire x1="63.43" y1="84.636196875" x2="63.5" y2="84.566196875" width="0.508" layer="1"/>
 <wire x1="63.5" y1="84.566196875" x2="62.553803125" y2="84.566196875" width="0.508" layer="1"/>
 <wire x1="61.189803125" y1="85.930196875" x2="57.970659375" y2="82.711053125" width="0.508" layer="1"/>
@@
 <contactref element="IC1" pad="45"/>
 <contactref element="U2" pad="24"/>
-<wire x1="25.67" y1="62.88013125" x2="25.6656" y2="62.87573125" width="0.254" layer="1"/>
-<wire x1="25.6656" y1="62.81400625" x2="25.6656" y2="62.87573125" width="0.254" layer="1"/>
-<wire x1="25.67" y1="62.5125" x2="25.67" y2="62.88013125" width="0.254" layer="1"/>
-<wire x1="25.6656" y1="62.87573125" x2="25.6656" y2="65.0356" width="0.2032" layer="1"/>
 <wire x1="25.6656" y1="65.0356" x2="26.67" y2="66.04" width="0.254" layer="1"/>
 <wire x1="26.67" y1="66.04" x2="33.02" y2="66.04" width="0.254" layer="1"/>
@@
 <wire x1="35.56" y1="49.53" x2="35.56" y2="51.3747375" width="0.2032" layer="1"/>
 <wire x1="35.56" y1="51.3747375" x2="34.29" y2="52.6447375" width="0.2032" layer="1"/>
+<wire x1="25.67" y1="62.5125" x2="25.67" y2="65.0312" width="0.254" layer="1"/>
+<wire x1="25.67" y1="65.0312" x2="25.6656" y2="65.0356" width="0.254" layer="1"/>
 </signal>
 <signal name="PB9">
