File: stm32f103_fc.brd (EAGLE design)
At the start: 53.1 x 76.5 mm, 49 parts, among them IC1 STM32F10XCXT6, IC2 LD1117AS33TR, U2 9DoF IMU, Y1 8MHz, Y2 32.768MHz

Commit message: version 2.0
Parts:
- removed C11, C13, C14, C7: 0.1uF, SparkFun-Capacitors:0402
- removed S1: SPST-SMD-5.2, SparkFun-Switches:TACTILE_SWITCH_SMD_5.2MM
- removed U2: 9DoF IMU, SparkFun-Sensors:QFN24-3X3
- added BUZZER: CMT-1285C-035, SparkFun-Electromechanical:BUZZER-12MM
- added C15, C22: 0.1uF, SparkFun-Capacitors:0402
- added C19: 2.2nF, SparkFun-Capacitors:0603
- added C23: 10nF, SparkFun-Capacitors:0603
- added IMU: MPU-6050, MPU-6050:QFN50P400X400X95-24N
- added SWITCH: MOMENTARY-SWITCH-SPST-SMD-4.5MM-轻触开关, SparkFun-Switches:TACTILE_SWITCH_SMD_4.5MM
- C18: device SparkFun-Capacitors:0603 -> SparkFun-Capacitors:0402
- C5: value 10nF -> 0.1uF; device SparkFun-Capacitors:0603 -> SparkFun-Capacitors:0402
- C6: device SparkFun-Capacitors:0402 -> SparkFun-Capacitors:0603
- HEADER: value (none) -> 2.54mm 2PX3P header
- IC1: value STM32F10XCXT6 -> STM32F103C8T6
- LED1, LED2: value GREEN -> BL-HGE36G-AV-TRB
- MICRO-USB: value (none) -> Micro-USB-5P-无柱-SMD
- N-CHANNEL-MOSFET, N-CHANNEL-MOSFET-2: value (none) -> 2N7002KT1G
- POWER_INPUT: value (none) -> KF350-2P-terminal-block-接线端子
- PY1, PY2: value 1X2-3.5MM -> 1X2-3.5MM KF350 terminal block
- R10, R13: value 22 -> 22omh
- R11, R9: value 680 -> 680omh
- R4, R5: value 470 -> 470omh
- SERVO_X, SERVO_Y: value (none) -> 2.54mm 3P header
- SWD: value (none) -> 2.54mm 4P header
- moved C18 95.9 mm to (-6.35, -29.5), turned to 0 degrees
- moved C5 89.1 mm to (-6.35, -26.2), turned to 0 degrees
- moved C6 84.2 mm to (-6.35, -22.9)
- renumbered D1 to LED1, D2 to LED2, J3 to MICRO-USB, Q1 to N-CHANNEL-MOSFET, Q2 to N-CHANNEL-MOSFET-2
Connections:
- removed net N$11: C6.2, U2.10
- removed net N$28: IC1.35
- removed net N$30: IC1.36
- removed net N$31: IC1.24
- removed net VBAT: IC1.1
- new net N$16: C22.2, IMU.10
- new net N$4: C19.1, IMU.20
- net 9V: now also C6.2; no longer MICRO-USB.VBUS
- net GND: now also BUZZER.-, C15.1, C18.1, C19.2, C22.1, C23.1, C4.2, C5.1, C8.2, IC1.35, IMU.1, IMU.11, IMU.18, SWITCH.2, SWITCH.3; no longer C11.2, C13.2, C14.2, C18.2, C5.2, C6.1, C7.2, S1.1, S1.2, U2.11, U2.18, U2.20
- net N$10: now also C6.1, MICRO-USB.VBUS; no longer C4.2, C8.2
- net PA12: no longer U2.12
- net PB0: now also IMU.12
- net PB1: now also BUZZER.+
- net PB8: now also IMU.24; no longer U2.24
- net PB9: now also IMU.23; no longer U2.23
- net RESET: now also SWITCH.1, SWITCH.4; no longer S1.3, S1.4
- net VCC3V3: now also C15.2, C18.2, C23.2, C5.2, IC1.1, IC1.24, IC1.36, IMU.13, IMU.8; no longer C11.1, C13.1, C14.1, C18.1, C5.1, C7.1, U2.1, U2.13, U2.22, U2.8
Routing:
- net GND: track 338.3 -> 259.1 mm, vias 19 -> 15
- net VCC3V3: track 230.2 -> 195.8 mm
- net RESET: track 41.0 -> 33.5 mm
- net N$11: track 5.01 -> 0.00 mm
- net 9V: track 167.3 -> 162.9 mm
- net N$10: track 3.38 -> 0.00 mm
- net PB8: track 31.0 -> 28.5 mm
- net PB9: track 28.7 -> 26.7 mm
- net PA12: track 55.5 -> 54.7 mm

Commit message: version 2.0 done
Parts:
- moved C18 101.7 mm to (49.9, 55.2)
- moved C5 101.4 mm to (49.9, 58.2)
- moved SWITCH 76.7 mm to (43.9, 25.8), turned to 180 degrees
- moved C19 73.1 mm to (30.0, 68.3), turned to 90 degrees
- moved C23 71.6 mm to (22.7, 53.3)
- moved C22 69.8 mm to (31.5, 51.9), flipped to the bottom, turned to 90 degrees
- moved IMU 68.4 mm to (28.7, 58.3)
- moved BUZZER 65.8 mm to (56.3, 18.4), turned to 90 degrees
- moved C6 51.5 mm to (24.0, 18.8), turned to 270 degrees
- moved C15 51.1 mm to (36.3, 46.4), turned to 180 degrees
- moved R10 40.8 mm to (45.3, 58.2), flipped to the bottom, turned to 0 degrees
- moved R3 0.51 mm to (31.2, 25.4)
Routing:
- net VCC3V3: track 195.8 -> 252.2 mm
- net N$6: track 12.4 -> 66.7 mm, vias 0 -> 5
- net PA11: track 51.8 -> 5.81 mm, vias 2 -> 1
- net PB1: track 0.00 -> 37.5 mm, vias 0 -> 1
- net PB0: track 0.00 -> 21.3 mm, vias 0 -> 2
- net GND: track 259.1 -> 239.0 mm, vias 15 -> 12
- net N$4: track 0.00 -> 11.2 mm, vias 0 -> 2
- net N$10: track 0.00 -> 8.44 mm
- net RESET: track 33.5 -> 39.8 mm
- net PB8: track 28.5 -> 34.0 mm
- net N$16: track 0.00 -> 5.27 mm, vias 0 -> 1
- net 9V: track 162.9 -> 165.4 mm
- net PB9: track 26.7 -> 28.6 mm
- net PA12: track 54.7 -> 56.3 mm, vias 2 -> 4
- removed copper zone on layer 1, net GND

Commit message: version 1.0.1 done
Routing:
- added copper zone on layer 1, net GND
Changed lines of the file:
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@@
 <wire x1="40.03" y1="83.13419375" x2="40.03" y2="81.0538625" width="0.508" layer="1"/>
 <wire x1="44.43" y1="46.28298125" x2="44.43" y2="46.2802625" width="0.2032" layer="1"/>
-<wire x1="44.43" y1="44.0838125" x2="44.43" y2="41.93" width="0.2032" layer="1"/>
+<wire x1="44.43" y1="44.0838125" x2="44.43" y2="43.688" width="0.2032" layer="1"/>
+<wire x1="44.43" y1="43.688" x2="44.43" y2="41.93" width="0.2032" layer="1"/>
 <wire x1="44.43" y1="41.93" x2="49.53" y2="36.83" width="0.2032" layer="1"/>
 <wire x1="44.43" y1="46.28298125" x2="44.43298125" y2="46.28" width="0.2032" layer="1"/>
@@
 <wire x1="35.742" y1="46.355" x2="33.4474" y2="46.355" width="0.2032" layer="1"/>
 <wire x1="33.4474" y1="46.355" x2="33.23" y2="46.5724" width="0.2032" layer="1"/>
-<wire x1="41.91" y1="13.97" x2="41.91" y2="13.716" width="0.2032" layer="1"/>
 <wire x1="40.43" y1="55.3" x2="40.43" y2="53.55" width="0.2032" layer="1"/>
 <wire x1="40.43" y1="53.55" x2="40.64" y2="53.34" width="0.2032" layer="1"/>
@@
 <wire x1="40.43" y1="48.05" x2="40.767" y2="48.387" width="0.2032" layer="1"/>
 <wire x1="40.767" y1="48.387" x2="43.688" y2="48.387" width="0.2032" layer="1"/>
-<wire x1="43.688" y1="48.387" x2="44.43" y2="47.645" width="0.2032" layer="1"/>
+<wire x1="44.43" y1="47.645" x2="43.688" y2="48.387" width="0.2032" layer="1"/>
 <wire x1="44.43" y1="46.3" x2="44.4302625" y2="46.2997375" width="0.2032" layer="1"/>
 <wire x1="44.4302625" y1="46.2997375" x2="44.4302625" y2="46.28" width="0.2032" layer="1"/>
-<wire x1="44.43" y1="46.3" x2="44.43" y2="45.43646875" width="0.2032" layer="1"/>
-<wire x1="44.43" y1="45.43646875" x2="45.106328125" y2="44.760140625" width="0.2032" layer="1"/>
-<wire x1="44.43" y1="47.645" x2="44.43" y2="46.3" width="0.2032" layer="1"/>
+<wire x1="44.43" y1="46.3" x2="44.43" y2="47.645" width="0.2032" layer="1"/>
+<wire x1="44.43" y1="46.3" x2="44.43" y2="44.0838125" width="0.2032" layer="1"/>
 </signal>
 <signal name="N$1">
@@
 <wire x1="28.499" y1="67.703" x2="29.972" y2="69.176" width="0.2032" layer="1"/>
 <wire x1="28.321" y1="76.2" x2="34.71" y2="76.2" width="0.508" layer="1"/>
-<wire x1="50.60064375" y1="53.05" x2="49.331" y2="55.245" width="0" layer="19" extent="1-1"/>
-<wire x1="40.93" y1="55.3" x2="47.68" y2="53.05" width="0" layer="19" extent="1-1"/>
-<wire x1="38.68" y1="48.55" x2="40.93" y2="55.3" width="0" layer="19" extent="1-1"/>
-<wire x1="36.902" y1="46.355" x2="38.68" y2="48.55" width="0" layer="19" extent="1-1"/>
-<wire x1="29.452" y1="56.323" x2="26.67" y2="53.34" width="0" layer="19" extent="1-1"/>
-<wire x1="30.672" y1="59.543" x2="29.452" y2="56.323" width="0" layer="19" extent="1-1"/>
-<wire x1="26.732" y1="59.543" x2="30.672" y2="59.543" width="0" layer="19" extent="1-1"/>
-<wire x1="31.75" y1="63.5" x2="30.672" y2="59.543" width="0" layer="19" extent="1-1"/>
-<wire x1="21.883" y1="53.34" x2="26.67" y2="53.34" width="0" layer="19" extent="1-1"/>
-<wire x1="28.499" y1="67.703" x2="31.75" y2="63.5" width="0" layer="19" extent="1-1"/>
-<wire x1="43.93" y1="46.3" x2="38.68" y2="48.55" width="0" layer="19" extent="1-1"/>
-<wire x1="46.167" y1="27.531" x2="48.87308125" y2="24.1875" width="0" layer="19" extent="1-1"/>
-<wire x1="41.717" y1="27.531" x2="46.167" y2="27.531" width="0" layer="19" extent="1-1"/>
-<wire x1="44.87" y1="33.02" x2="48.87308125" y2="36.791665625" width="0" layer="19" extent="1-1"/>
-<wire x1="56.261" y1="15.165" x2="46.99" y2="13.97" width="0" layer="19" extent="1-1"/>
+<polygon width="0.2032" layer="1">
+<vertex x="14.097" y="91.059"/>
+<vertex x="75.438" y="91.059"/>
+<vertex x="75.819" y="91.44"/>
+<vertex x="75.819" y="9.398"/>
+<vertex x="74.295" y="7.874"/>
+<vertex x="15.621" y="7.874"/>
+<vertex x="14.224" y="9.271"/>
+<vertex x="14.097" y="9.398"/>
+</polygon>
 </signal>
 <signal name="N$3">
@@
 <contactref element="R10" pad="2"/>
 <contactref element="IC1" pad="32"/>
-<wire x1="42.41035" y1="55.31965" x2="42.43" y2="55.3" width="0.2032" layer="1"/>
 <wire x1="42.43" y1="55.3" x2="42.43" y2="58.774" width="0.2032" layer="1"/>
 <wire x1="43.038" y1="58.166" x2="44.489" y2="58.166" width="0.2032" layer="16"/>
