File: stm32f103_fc.sch (EAGLE design)
At the start: 47 parts, among them IC1 STM32F10XCXT6, IC2 LD1117AS33TR, U2 9DoF IMU, Y1 8MHz, Y2 32.768MHz

Commit message: change all width to 8mil
Parts:
- renumbered PYRO1 to PY1, PYRO2 to PY2
Changed lines of the file:
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@@
 <part name="GND28" library="SparkFun-PowerSymbols" library_urn="urn:adsk.eagle:library:530" deviceset="GND" device=""/>
 <part name="POWER_INPUT" library="SparkFun-Connectors" library_urn="urn:adsk.eagle:library:513" deviceset="CONN_02" device="3.5MM" package3d_urn="urn:adsk.eagle:package:38050/1"/>
-<part name="PYRO1" library="adafruit" library_urn="urn:adsk.eagle:library:420" deviceset="1X2" device="-3.5MM" package3d_urn="urn:adsk.eagle:package:6240635/1"/>
+<part name="PY1" library="adafruit" library_urn="urn:adsk.eagle:library:420" deviceset="1X2" device="-3.5MM" package3d_urn="urn:adsk.eagle:package:6240635/1"/>
 <part name="Q1" library="adafruit" library_urn="urn:adsk.eagle:library:420" deviceset="MOSFET-N" device="REFLOW" package3d_urn="urn:adsk.eagle:package:6240836/1"/>
 <part name="GND31" library="SparkFun-PowerSymbols" library_urn="urn:adsk.eagle:library:530" deviceset="GND" device=""/>
-<part name="PYRO2" library="adafruit" library_urn="urn:adsk.eagle:library:420" deviceset="1X2" device="-3.5MM" package3d_urn="urn:adsk.eagle:package:6240635/1"/>
+<part name="PY2" library="adafruit" library_urn="urn:adsk.eagle:library:420" deviceset="1X2" device="-3.5MM" package3d_urn="urn:adsk.eagle:package:6240635/1"/>
 <part name="Q2" library="adafruit" library_urn="urn:adsk.eagle:library:420" deviceset="MOSFET-N" device="REFLOW" package3d_urn="urn:adsk.eagle:package:6240836/1"/>
 <part name="GND30" library="SparkFun-PowerSymbols" library_urn="urn:adsk.eagle:library:530" deviceset="GND" device=""/>
@@
 <attribute name="NAME" x="-66.04" y="124.968" size="1.778" layer="95" font="vector"/>
 </instance>
-<instance part="PYRO1" gate="G$1" x="-25.4" y="190.5" smashed="yes"/>
+<instance part="PY1" gate="G$1" x="-25.4" y="190.5" smashed="yes"/>
 <instance part="Q1" gate="G$1" x="-53.34" y="182.88" smashed="yes">
 <attribute name="NAME" x="-48.26" y="183.515" size="1.27" layer="95"/>
@@
 <attribute name="VALUE" x="-50.8" y="172.466" size="1.778" layer="96" align="top-center"/>
 </instance>
-<instance part="PYRO2" gate="G$1" x="33.02" y="190.5" smashed="yes"/>
+<instance part="PY2" gate="G$1" x="33.02" y="190.5" smashed="yes"/>
 <instance part="Q2" gate="G$1" x="5.08" y="182.88" smashed="yes">
 <attribute name="NAME" x="10.16" y="183.515" size="1.27" layer="95"/>
@@
 </segment>
 <segment>
-<pinref part="PYRO1" gate="G$1" pin="1"/>
+<pinref part="PY1" gate="G$1" pin="1"/>
 <wire x1="-30.48" y1="193.04" x2="-50.8" y2="193.04" width="0.1524" layer="91"/>
 <label x="-50.8" y="193.04" size="1.778" layer="95"/>
 </segment>
 <segment>
-<pinref part="PYRO2" gate="G$1" pin="1"/>
+<pinref part="PY2" gate="G$1" pin="1"/>
 <wire x1="27.94" y1="193.04" x2="7.62" y2="193.04" width="0.1524" layer="91"/>
 <label x="7.62" y="193.04" size="1.778" layer="95"/>
@@
 <net name="N$14" class="0">
 <segment>
-<pinref part="PYRO1" gate="G$1" pin="2"/>
+<pinref part="PY1" gate="G$1" pin="2"/>
 <wire x1="-30.48" y1="190.5" x2="-35.56" y2="190.5" width="0.1524" layer="91"/>
 <pinref part="R12" gate="G$1" pin="2"/>
@@
 <net name="N$12" class="0">
 <segment>
-<pinref part="PYRO2" gate="G$1" pin="2"/>
+<pinref part="PY2" gate="G$1" pin="2"/>
 <wire x1="27.94" y1="190.5" x2="22.86" y2="190.5" width="0.1524" layer="91"/>
 <pinref part="R15" gate="G$1" pin="2"/>
